File: pcb/opaque-r2/opaque-r2.kicad_sch (KiCad schematic)
At the start: 15 parts, among them J1 Conn_01x01_Socket, J2 Conn_01x02_Pin, J3 Conn_01x02_Pin, J4 Conn_01x02_Pin, J5 Conn_01x02_Pin, U1 ESP32-DevKitC

Commit message: Writtin code
Other:
- added sheet Power (power.kicad_sch)
Changed lines of the file:
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@@
 		)
 		(property "Value" "GND"
-			(at 67.31 149.352 90)
+			(at 69.088 149.606 0)
 			(effects
 				(font
@@
 	)
 	(sheet
+		(at 189.23 25.4)
+		(size 26.67 10.16)
+		(fields_autoplaced yes)
+		(stroke
+			(width 0.1524)
+			(type solid)
+		)
+		(fill
+			(color 0 0 0 0.0000)
+		)
+		(property "Sheetname" "5V Parts"
+			(at 189.23 24.6884 0)
+			(effects
+				(font
+					(size 1.27 1.27)
+				)
+				(justify left bottom)
+			)
+		)
+		(property "Sheetfile" "5V_parts.kicad_sch"
+			(at 189.23 36.1446 0)
+			(effects
+				(font
+					(size 1.27 1.27)
+				)
+				(justify left top)
+			)
+		)
+		(instances
+			(project "opaque-r2"
+				(path "/7438ae78-2675-47f2-b3a6-7b20cbf2e31f"
+					(page "2")
+				)
+			)
+		)
+	)
+	(sheet
 		(at 158.75 25.4)
 		(size 26.67 10.16)
@@
 			(color 0 0 0 0.0000)
 		)
-		(property "Sheetname" "5V Parts"
+		(property "Sheetname" "Power"
 			(at 158.75 24.6884 0)
 			(effects
@@
 			)
 		)
-		(property "Sheetfile" "5V_parts.kicad_sch"
+		(property "Sheetfile" "power.kicad_sch"
 			(at 158.75 36.1446 0)
 			(effects
@@
 			(project "opaque-r2"
 				(path "/7438ae78-2675-47f2-b3a6-7b20cbf2e31f"
-					(page "2")
-				)
-			)
+					(page "3")
+				)
+			)
