File: Hardware/pcb/opaque-v2.01/5V_parts.kicad_sch (KiCad schematic)
At the start: 14 parts

Commit message: Changed more
Other:
- company: (none) -> Barkın Özsoy (barkolorious)
- title: Açık-kaynaklı Taşınabilir Hava Kalitesi Ölçüm Kitleri -> opaque: Open-source Portable Air QUality Equipment
Changed lines of the file:
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@@
 (kicad_sch
-	(version 20231120)
+	(version 20250114)
 	(generator "eeschema")
-	(generator_version "8.0")
+	(generator_version "9.0")
 	(paper "A4")
 	(title_block
-		(title "Açık-kaynaklı Taşınabilir Hava Kalitesi Ölçüm Kitleri")
+		(title "opaque: Open-source Portable Air QUality Equipment")
 		(date "2025-02-01")
-		(rev "R1.1")
-		(comment 1 "TÜBİTAK 2204-D")
+		(rev "R2.1")
+		(company "Barkın Özsoy (barkolorious)")
+		(comment 1 "TÜBİTAK 2204-D Lise Öğrencileri İklim Değişikliği Araştırma Projeleri Yarışmaları")
 	)
 	(junction
