File: Hardware/pcb/opaque-v2.01/opaque-v2.01.kicad_sch (KiCad schematic)
At the start: 15 parts, among them J1 Conn_01x01_Socket, J2 Conn_01x02_Pin, J3 Conn_01x02_Pin, J4 Conn_01x02_Pin, J5 Conn_01x02_Pin, U1 ESP32-DevKitC

Commit message: Changed more
Changed lines of the file:
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@@
 (kicad_sch
-	(version 20231120)
+	(version 20250114)
 	(generator "eeschema")
-	(generator_version "8.0")
+	(generator_version "9.0")
 	(paper "A4")
 	(title_block
 		(title "opaque: Open-source Portable Air QUality Equipment")
 		(date "2025-02-01")
-		(rev "R1.1")
+		(rev "R2.1")
 		(company "Barkın Özsoy (barkolorious)")
-		(comment 1 "TÜBİTAK 2204-A")
+		(comment 1 "TÜBİTAK 2204-D Lise Öğrencileri İklim Değişikliği Araştırma Projeleri Yarışmaları")
 	)
 	(junction
@@
 		(at 189.23 25.4)
 		(size 26.67 10.16)
+		(exclude_from_sim no)
+		(in_bom yes)
+		(on_board yes)
+		(dnp no)
 		(fields_autoplaced yes)
 		(stroke
@@
 		)
 		(instances
-			(project "opaque-r2"
+			(project "opaque-v2.01"
 				(path "/7438ae78-2675-47f2-b3a6-7b20cbf2e31f"
 					(page "2")
@@
 		(at 158.75 25.4)
 		(size 26.67 10.16)
+		(exclude_from_sim no)
+		(in_bom yes)
+		(on_board yes)
+		(dnp no)
 		(fields_autoplaced yes)
 		(stroke
@@
 		)
 		(instances
-			(project "opaque-r2"
+			(project "opaque-v2.01"
 				(path "/7438ae78-2675-47f2-b3a6-7b20cbf2e31f"
 					(page "3")
@@
 		)
 	)
+	(embedded_fonts no)
 )
